File: tensigral_lamp_hardware/tensigral_lamp_hardware.kicad_pcb (KiCad board)
At the start: 2 copper layers, 99.5 x 99.8 mm, 37 parts, among them J1 USB_B_Micro, P1 CONN_1, P2 CONN_1, P3 CONN_1, P4 CONN_1, P5 CONN_1, P6 CONN_1, U1 STM32F042F4Px

Commit message: update
Parts:
- added C10: 22uF, Capacitor_SMD:C_0805_2012Metric_Pad1.15x1.40mm_HandSolder, F.Cu at (81.2, 47.8)
- added C11: 22nF, Capacitor_SMD:C_0805_2012Metric_Pad1.15x1.40mm_HandSolder, F.Cu at (43.1, 83.2)
- added C12: 22uF, Capacitor_SMD:C_0805_2012Metric_Pad1.15x1.40mm_HandSolder, F.Cu at (55.2, 74.2)
- added C13: 22uF, Capacitor_SMD:C_0805_2012Metric_Pad1.15x1.40mm_HandSolder, F.Cu at (42.8, 77.0)
- added C14: 22nF, Capacitor_SMD:C_0805_2012Metric_Pad1.15x1.40mm_HandSolder, F.Cu at (46.8, 87.8)
- added C15: 22nF, Capacitor_SMD:C_0805_2012Metric_Pad1.15x1.40mm_HandSolder, F.Cu at (57.9, 71.2)
- added C16: 22uF, Capacitor_SMD:C_0805_2012Metric_Pad1.15x1.40mm_HandSolder, F.Cu at (87.7, 39.8)
- added C17: 22nF, Capacitor_SMD:C_0805_2012Metric_Pad1.15x1.40mm_HandSolder, F.Cu at (107.8, 43.6)
- added J2: JTAG, kicad:RIBBON6SMT_POGO_OR_IDC, F.Cu at (65.5, 71.0)
- added J3: EXTCTL, kicad:RIBBON6SMT_POGO_OR_IDC, F.Cu at (72.0, 57.5)
- added J4: WSOUT, Connector_PinHeader_2.54mm:PinHeader_1x03_P2.54mm_Vertical, F.Cu at (76.2, 76.2)
- added J5: AVRISP6, kicad:RIBBON6SMT_POGO_OR_IDC, F.Cu at (78.2, 34.9)
- added L1: 10uH, Inductor_SMD:L_2816_7142Metric, F.Cu at (49.5, 79.0)
- added MK1: Microphone, kicad:9mmELECTRET_MIC_SMT, F.Cu at (48.2, 42.4)
- added P10: AUXOUT, Connector_Wire:SolderWirePad_1x01_Drill1mm, F.Cu at (106.9, 82.4)
- added P11: AUXEXTRA, Connector_Wire:SolderWirePad_1x01_Drill1mm, F.Cu at (65.0, 35.5)
- added P7: AUX, Connector_Wire:SolderWirePad_1x01_Drill0.8mm, F.Cu at (82.8, 70.3)
- added P8: WS, Connector_Wire:SolderWirePad_1x01_Drill0.8mm, F.Cu at (88.5, 62.0)
- added P9: AUXOUT, Connector_Wire:SolderWirePad_1x01_Drill1mm, F.Cu at (109.5, 76.2)
- added R1: 33k,1%, Resistor_SMD:R_0805_2012Metric_Pad1.15x1.40mm_HandSolder, F.Cu at (39.2, 91.2)
- added R2: 6.8k,1%, Resistor_SMD:R_0805_2012Metric_Pad1.15x1.40mm_HandSolder, F.Cu at (38.2, 87.2)
- added R3: 6.8k,1%, Resistor_SMD:R_0805_2012Metric_Pad1.15x1.40mm_HandSolder, F.Cu at (38.9, 54.1)
- added R4: 6.8k,1%, Resistor_SMD:R_0805_2012Metric_Pad1.15x1.40mm_HandSolder, F.Cu at (103.2, 48.2)
- added R5: 6.8k,1%, Resistor_SMD:R_0805_2012Metric_Pad1.15x1.40mm_HandSolder, F.Cu at (104.1, 41.9)
- added R6: 6.8k,1%, Resistor_SMD:R_0805_2012Metric_Pad1.15x1.40mm_HandSolder, F.Cu at (29.8, 36.2)
- added SW1: TACTILE, kicad:TACTILE10B, F.Cu at (33.7, 47.2)
- added T0: TOUCH0, kicad:TOUCH_MARK, F.Cu at (31.8, 84.8)
- added T1: TOUCH1, kicad:TOUCH_MARK, F.Cu at (40.6, 35.5)
- added T2: TOUCH2, kicad:TOUCH_MARK, F.Cu at (82.8, 58.4)
- added U2: MT2492, Package_TO_SOT_SMD:SOT-23-6_Handsoldering, F.Cu at (43.0, 86.3)
- added U3: ATtiny85-20SU, Package_SO:SOIJ-8_5.3x5.3mm_P1.27mm, F.Cu at (96.7, 41.1)
- added U4: MXC400xXC, kicad:MXC400xXC, F.Cu at (105.0, 44.8)
- C1, C2, C3, C4, C5, C6, C7, C8, C9: value .1uF -> 22nF
- D1, D10, D11, D12, D13, D14, D15, D16, D17, D18, D19, D2, D20, D3, D4, D5, D6, D7, D8, D9: value WS2812B -> SK6812W
- P1: value CONN_1 -> WSIN; footprint Connector_Wire:SolderWirePad_1x01_Drill0.8mm -> Connector_Wire:SolderWirePad_1x01_Drill1mm
- P2: value CONN_1 -> WSOUT; footprint Connector_Wire:SolderWirePad_1x01_Drill0.8mm -> Connector_Wire:SolderWirePad_1x01_Drill1mm
- P3, P4: value CONN_1 -> VLED; footprint Connector_Wire:SolderWirePad_1x01_Drill0.8mm -> Connector_Wire:SolderWirePad_1x01_Drill1mm
- P5, P6: value CONN_1 -> GND; footprint Connector_Wire:SolderWirePad_1x01_Drill0.8mm -> Connector_Wire:SolderWirePad_1x01_Drill1mm
- moved C6 32.7 mm to (93.0, 77.7), turned to 315 degrees
- moved C9 21.5 mm to (55.2, 60.5), turned to 90 degrees
- moved U1 8.65 mm to (60.9, 61.1), turned to 190 degrees
- moved D12 0.36 mm to (20.1, 86.8), turned to 258 degrees
- turned C5 to 70 degrees
- turned D15 to 280 degrees
- turned D17 to 175 degrees
- turned D18 to 140 degrees
Connections:
- C1 pad 1: +5V -> VLED
- C2 pad 1: +5V -> VLED
- C3 pad 1: +5V -> VLED
- C4 pad 1: +5V -> VLED
- C5 pad 1: +5V -> VLED
- C6 pad 1: +5V -> VLED
- C7 pad 1: +5V -> VLED
- C8 pad 1: +5V -> VLED
- C9 pad 1: +5V -> +3V8
- D1 pad 1: +5V -> VLED
- D10 pad 1: +5V -> VLED
- D11 pad 1: +5V -> VLED
- D12 pad 1: +5V -> VLED
- D13 pad 1: +5V -> VLED
- D14 pad 1: +5V -> VLED
- D15 pad 1: +5V -> VLED
- D16 pad 1: +5V -> VLED
- D17 pad 1: +5V -> VLED
- D18 pad 1: +5V -> VLED
- D19 pad 1: +5V -> VLED
- D2 pad 1: +5V -> VLED
- D20 pad 1: +5V -> VLED
- D3 pad 1: +5V -> VLED
- D4 pad 1: +5V -> VLED
- D5 pad 1: +5V -> VLED
- D6 pad 1: +5V -> VLED
- D7 pad 1: +5V -> VLED
- D8 pad 1: +5V -> VLED
- D9 pad 1: +5V -> VLED
- J1 pad 1: (no net) -> VUSB
- J1 pad 2: (no net) -> D-
- J1 pad 3: (no net) -> D+
- P2 pad 1: WS2812U -> WS2812UM
- P3 pad 1: +5V -> VLED
- P4 pad 1: +5V -> +3V8
- U1 pad 1: (no net) -> Net-(R3-Pad2)
- U1 pad 10: (no net) -> PA4
- U1 pad 11: (no net) -> PA5
- U1 pad 12: (no net) -> PA6
- U1 pad 13: (no net) -> WS2812U
- U1 pad 14: (no net) -> AUX
- U1 pad 16: (no net) -> +3V8
- U1 pad 17: (no net) -> D-
- U1 pad 18: (no net) -> D+
- U1 pad 19: (no net) -> SWD
- U1 pad 2: (no net) -> PF0
- U1 pad 20: (no net) -> SWC
- U1 pad 3: (no net) -> PF1
- U1 pad 4: (no net) -> NRST
- U1 pad 5: (no net) -> +3V8
- U1 pad 6: WS2812U -> Net-(T0-Pad1)
- U1 pad 7: (no net) -> Net-(T1-Pad1)
- U1 pad 8: (no net) -> ANA_ADC
- U1 pad 9: (no net) -> Net-(T2-Pad1)
Routing:
- net GND: track 0.00 -> 549.0 mm, vias 0 -> 14
- net VLED: track 0.00 -> 288.0 mm
- net VUSB: track 0.00 -> 130.6 mm, vias 0 -> 5
- net +3V8: track 0.00 -> 107.9 mm, vias 0 -> 4
- net WS2812U: track 0.00 -> 76.4 mm, vias 0 -> 2
- net AUXU: track 0.00 -> 71.8 mm, vias 0 -> 1
- net AUXGND: track 0.00 -> 69.8 mm, vias 0 -> 6
- net ANA_ADC: track 0.00 -> 56.9 mm
- net AUXVCC: track 0.00 -> 56.3 mm, vias 0 -> 3
- net Net-(T0-Pad1): track 0.00 -> 55.7 mm, vias 0 -> 4
- net AUX: track 0.00 -> 51.7 mm, vias 0 -> 2
- net Net-(R3-Pad2): track 0.00 -> 47.0 mm, vias 0 -> 2
- net Net-(T1-Pad1): track 0.00 -> 36.3 mm
- net AUXEXTRA: track 0.00 -> 30.2 mm
- net Net-(T2-Pad1): track 0.00 -> 26.9 mm
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- added copper zone on B.Cu, net (none)
- added copper zone on F.Cu, net (none)
- added copper zone on F.Cu, net AUX
- added copper zone on B.Cu, net AUXGND
- added copper zone on F.Cu, net AUXGND
- added copper zone on B.Cu, net AUXU
- added copper zone on F.Cu, net AUXU
- added copper zone on B.Cu, net AUXVCC
- added copper zone on F.Cu, net AUXVCC
- added copper zone on B.Cu, net GND
- added copper zone on F.Cu, net GND
- added copper zone on F.Cu, net VLED
- added copper zone on F.Cu, net WS2812U
- added copper zone on B.Cu, net WS2812UM
- added copper zone on F.Cu, net WS2812UM
Other:
- outline, holes or cut-outs redrawn
- net class Default: clearance 0.2 -> 0.199; trace_width 0.25 -> 0.3
- rule trace_clearance: 0.2 -> 0.199
- rule trace_min: 0.2 -> 0.3
- board text added: "+"
- board text added: "-"
- board text added: "AUX"
- board text added: "GND"
- board text added: "SWD +5 SWC NC RST 0V"
- board text added: "VLED"
- board text added: "WS"
- board text added: "tensigral_lamp r - https://github.com/cnlohr/tensigral_lamp"

Commit message: bump
Parts:
- D1, D10, D11, D12, D13, D14, D15, D16, D17, D18, D19, D2, D20, D3, D4, D5, D6, D7, D8, D9: value SK6812W -> SK6812-RGBWW
- J1: footprint Connector_USB:USB_Micro-B_Molex_47346-0001 -> kicad:USBMicroB-U253-051T-4BH89-F1B
- R1: value 33k,1% -> 33k-1%
- R2, R3, R4, R5, R6: value 6.8k,1% -> 6.8k-1%
- U3: value ATtiny85-20SU -> ATtiny45-20SU
- moved J1 1.50 mm to (35.4, 70.9), turned to 226 degrees
Routing:
- net GND: track 549.0 -> 544.1 mm
Other:
- board text added: "0V RST MO SK 4V MI"
- board text added: "PA4 PF1 PA5 PF0 PA6 GND"
