File: tensigral_lamp_hardware/tensigral_lamp_hardware.sch (KiCad schematic (older format))
At the start: 37 parts, among them J1 USB_B_Micro, P1 CONN_1, P2 CONN_1, P3 CONN_1, P4 CONN_1, P5 CONN_1, P6 CONN_1, U1 STM32F042F4Px

Commit message: update
Parts:
- added C10, C12, C13, C16: 22uF, Capacitor_SMD:C_0805_2012Metric_Pad1.15x1.40mm_HandSolder, symbol Device:C
- added C11, C14, C15, C17: 22nF, Capacitor_SMD:C_0805_2012Metric_Pad1.15x1.40mm_HandSolder, symbol Device:C
- added J2: JTAG, kicad:RIBBON6SMT_POGO_OR_IDC, symbol Connector_Generic:Conn_02x03_Odd_Even
- added J3: EXTCTL, kicad:RIBBON6SMT_POGO_OR_IDC, symbol Connector_Generic:Conn_02x03_Odd_Even
- added J4: WSOUT, Connector_PinHeader_2.54mm:PinHeader_1x03_P2.54mm_Vertical, symbol Connector_Generic:Conn_01x03
- added J5: AVRISP6, kicad:RIBBON6SMT_POGO_OR_IDC, symbol 5050RGB:AVRISP6
- added L1: 10uH, Inductor_SMD:L_2816_7142Metric, symbol Device:L
- added MK1: Microphone, kicad:9mmELECTRET_MIC_SMT, symbol Device:Microphone
- added P10, P9: AUXOUT, Connector_Wire:SolderWirePad_1x01_Drill1mm, symbol 5050RGB:CONN_1
- added P11: AUXEXTRA, Connector_Wire:SolderWirePad_1x01_Drill1mm, symbol 5050RGB:CONN_1
- added P7: AUX, Connector_Wire:SolderWirePad_1x01_Drill0.8mm, symbol 5050RGB:CONN_1
- added P8: WS, Connector_Wire:SolderWirePad_1x01_Drill0.8mm, symbol 5050RGB:CONN_1
- added R1: 33k,1%, Resistor_SMD:R_0805_2012Metric_Pad1.15x1.40mm_HandSolder, symbol Device:R
- added R2, R3, R4, R5, R6: 6.8k,1%, Resistor_SMD:R_0805_2012Metric_Pad1.15x1.40mm_HandSolder, symbol Device:R
- added SW1: TACTILE, kicad:TACTILE10B, symbol tactile:TACTILE
- added T0: TOUCH0, kicad:TOUCH_MARK, symbol 5050RGB:CONN_1
- added T1: TOUCH1, kicad:TOUCH_MARK, symbol 5050RGB:CONN_1
- added T2: TOUCH2, kicad:TOUCH_MARK, symbol 5050RGB:CONN_1
- added U2: MT2492, Package_TO_SOT_SMD:SOT-23-6_Handsoldering, symbol MT2492:MT2492
- added U3: ATtiny85-20SU, Package_SO:SOIJ-8_5.3x5.3mm_P1.27mm, symbol MCU_Microchip_ATtiny:ATtiny85-20SU
- added U4: MXC400xXC, kicad:MXC400xXC, symbol kicad:MXC400xXC
- C1, C2, C3, C4, C5, C6, C7, C8, C9: value .1uF -> 22nF; Cost100 0.004845 -> 0.003738; LCSC https://lcsc.com/product-detail/Multilayer-Ceramic-Capacitors-MLCC-SMD-SMT_CT41G-0805-2X1-50V-0-1mF-K-N_C126469.html -> https://lcsc.com/product-detail/Multilayer-Ceramic-Capacitors-MLCC-SMD-SMT_Walsin-Tech-Corp-0805B223K500_C123617.html
- D1, D10, D11, D12, D13, D14, D15, D16, D17, D18, D19, D2, D20, D3, D4, D5, D6, D7, D8, D9: value WS2812B -> SK6812W
- P1: value CONN_1 -> WSIN; footprint Connector_Wire:SolderWirePad_1x01_Drill0.8mm -> Connector_Wire:SolderWirePad_1x01_Drill1mm
- P2: value CONN_1 -> WSOUT; footprint Connector_Wire:SolderWirePad_1x01_Drill0.8mm -> Connector_Wire:SolderWirePad_1x01_Drill1mm
- P3, P4: value CONN_1 -> VLED; footprint Connector_Wire:SolderWirePad_1x01_Drill0.8mm -> Connector_Wire:SolderWirePad_1x01_Drill1mm
- P5, P6: value CONN_1 -> GND; footprint Connector_Wire:SolderWirePad_1x01_Drill0.8mm -> Connector_Wire:SolderWirePad_1x01_Drill1mm
Connections:
- net +3V8: now also P4.1, C12.1, L1.2, R1.2, R6.2, SW1.1
- net GND: now also C10.2, C12.2, C13.2, C14.2, C15.2, J2.6 (Pin_6), J3.6 (Pin_6), J4.3 (Pin_3), MK1.1 (-), R2.1, R3.1, U2.2 (GND)
- net WS2812U: now also J4.2 (Pin_2), P8.1; no longer P2.1
- net at U1.1 (PB8): now also R3.2, SW1.4
- net PA4: now reaches U1.10 (PA4)
- net PA4: now also J3.1 (Pin_1)
- net PA5: now reaches U1.11 (PA5)
- net PA5: now also J3.3 (Pin_3)
- net PA6: now reaches U1.12 (PA6)
- net PA6: now also J3.5 (Pin_5)
- net AUX: now reaches U1.14 (PB1)
- net AUX: now also P7.1
- net SWD: now reaches U1.19 (PA13)
- net SWD: now also J2.1 (Pin_1)
- net PF0: now reaches U1.2 (PF0)
- net PF0: now also J3.4 (Pin_4)
- net SWC: now reaches U1.20 (PA14)
- net SWC: now also J2.3 (Pin_3)
- net PF1: now reaches U1.3 (PF1)
- net PF1: now also J3.2 (Pin_2)
- net NRST: now reaches U1.4 (NRST)
- net NRST: now also C15.1, J2.5 (Pin_5)
- net at U1.6 (PA0): now also T0.1
- net at U1.7 (PA1): now also T1.1
- net ANA_ADC: now reaches U1.8 (PA2)
- net ANA_ADC: now also MK1.2 (+), R6.1
- net at U1.9 (PA3): now also T2.1
- net +5V renamed VLED
- net VLED: now also C10.1; no longer J1.1 (VBUS), P4.1
- new net: C11.1, U2.1 (BS)
- new net: R1.1, R2.2, U2.3 (FB)
- new net: C11.2, L1.1, U2.6 (SW)
- new net: J5.5 (RST), U3.1 (~RESET~/PB5)
- new net: J5.1 (MISO), U3.6 (PB1)
- new net: J5.3 (SCK), U3.7 (PB2)
- new net ASCL: R5.2, U3.3 (XTAL2/PB4), U4.1 (SCL)
- new net ASDA: R4.1, U3.2 (XTAL1/PB3), U4.5 (SDA)
- new net AUXEXTRA: J5.4 (MOSI), P11.1, U3.5 (AREF/PB0)
- new net AUXGND: C16.2, C17.2, J5.6 (GND), U3.4 (GND), U4.3 (GND)
- new net AUXU: P10.1, P9.1
- new net AUXVCC: C16.1, C17.1, J5.2 (VCC), R4.2, R5.1, U3.8 (VCC), U4.6 (VDD)
- new net VUSB: C13.1, C14.1, J1.1 (VBUS), J2.2 (Pin_2), J4.1 (Pin_1), U2.4 (EN), U2.5 (IN)
- new net WS2812UM: P2.1
- no-connect marks 0 -> 2
Other:
- note added: "No external matching impedance needed.\nDriver contains matching impedance."
- moved on the sheet: D1, D17, D18, D19, D2, D20, D3, J1, P2, P3, P4, P5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

Commit message: bump
Parts:
- D1, D10, D11, D12, D13, D14, D15, D16, D17, D18, D19, D2, D20, D3, D4, D5, D6, D7, D8, D9: value SK6812W -> SK6812-RGBWW; Cost100 (none) -> .112; LCSC (none) -> https://www.aliexpress.com/item/32814778563.html
- J1: footprint Connector_USB:USB_Micro-B_Molex_47346-0001 -> kicad:USBMicroB-U253-051T-4BH89-F1B; Cost100 (none) -> .037085; LCSC (none) -> https://lcsc.com/product-detail/USB-Connectors_XKB-Enterpri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
- J2, J3: Cost100 (none) -> 0.024623; Cost1000 0.024623 -> (none)
- J4, P1, P10, P11, P2, P3, P4, P5, P6, P7, P8, P9, T0, T1, T2: NOBOM (none) -> 1
- J5: Cost100 (none) -> .042632; LCSC (none) -> https://lcsc.com/product-detail/Pin-Header-Female-Header_Ck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
- L1: Cost100 (none) -> 0.028295; Cost1000 0.028295 -> (none)
- MK1: Cost100 (none) -> 0.075806; Cost1000 0.075806 -> (none)
- R1: value 33k,1% -> 33k-1%; Cost100 (none) -> 0.001004; Cost1000 0.001004 -> (none)
- R2, R3, R4, R5, R6: value 6.8k,1% -> 6.8k-1%; Cost100 (none) -> .00104; Cost1000 .00104 -> (none)
- SW1: Cost100 (none) -> 0.007906; Cost1000 0.007906 -> (none)
- U1: Cost100 (none) -> 0.822727; LCSC (none) -> https://lcsc.com/product-detail/ST-Microelectronics_STMicro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
- U2: Cost100 (none) -> .053488; Cost1000 .053488 -> (none)
- U3: value ATtiny85-20SU -> ATtiny45-20SU; Cost100 (none) -> .837879; LCSC (none) -> https://lcsc.com/product-detail/MICROCHIP_MICROCHIP_ATTINY4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
- U4: Cost100 (none) -> 0.184848; Cost1000 0.184848 -> (none)

Commit message: Bump - fixing incorrect button part.
Parts:
- C1, C10, C11, C12, C13, C14, C15, C16, C17, C2, C3, C4, C5, C6, C7, C8, C9: symbol Device:C -> tensigral_lamp_hardware-rescue:C-Device
- D1, D10, D11, D12, D13, D14, D15, D16, D17, D18, D19, D2, D20, D3, D4, D5, D6, D7, D8, D9: symbol LED:WS2812B -> tensigral_lamp_hardware-rescue:WS2812B-LED
- J1: symbol Connector:USB_B_Micro -> tensigral_lamp_hardware-rescue:USB_B_Micro-Connector
- J2, J3: symbol Connector_Generic:Conn_02x03_Odd_Even -> tensigral_lamp_hardware-rescue:Conn_02x03_Odd_Even-Connector_Generic
- J4: symbol Connector_Generic:Conn_01x03 -> tensigral_lamp_hardware-rescue:Conn_01x03-Connector_Generic
- J5: symbol 5050RGB:AVRISP6 -> tensigral_lamp_hardware-rescue:AVRISP6-5050RGB
- L1: symbol Device:L -> tensigral_lamp_hardware-rescue:L-Device
- MK1: symbol Device:Microphone -> tensigral_lamp_hardware-rescue:Microphone-Device
- P1, P10, P11, P2, P3, P4, P5, P6, P7, P8, P9, T0, T1, T2: symbol 5050RGB:CONN_1 -> tensigral_lamp_hardware-rescue:CONN_1-5050RGB
- R1, R2, R3, R4, R5, R6: symbol Device:R -> tensigral_lamp_hardware-rescue:R-Device
- SW1: symbol tactile:TACTILE -> tensigral_lamp_hardware-rescue:TACTILE-tactile; Cost100 0.007906 -> 0.01388; LCSC https://lcsc.com/product-detail/Tactile-Switches_BOOMELE-Bo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 -> https://lcsc.com/product-detail/Tactile-Switches_SHOU-HAN-T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
- U1: symbol MCU_ST_STM32F0:STM32F042F4Px -> tensigral_lamp_hardware-rescue:STM32F042F4Px-MCU_ST_STM32F0
- U2: symbol MT2492:MT2492 -> tensigral_lamp_hardware-rescue:MT2492-MT2492
- U3: symbol MCU_Microchip_ATtiny:ATtiny85-20SU -> tensigral_lamp_hardware-rescue:ATtiny85-20SU-MCU_Microchip_ATtiny
- U4: symbol kicad:MXC400xXC -> tensigral_lamp_hardware-rescue:MXC400xXC-kicad
