File: attic/old_tensigral_lamp_2/tensigral_lamp_hardware.kicad_pcb (KiCad board)
At the start: 2 copper layers, 99 x 99.8 mm, 75 parts, among them J1 USB_B_Micro, J2 JTAG, J4 WSOUT, J6 MICJ, J8 WS_SEL, P1 WSIN, P10 AUXTOUCH, P2 WSOUT, P3 VLED, P4 VLED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

Commit message: Bump
Parts:
- removed C20: 22nF, Capacitor_SMD:C_0805_2012Metric_Pad1.15x1.40mm_HandSolder
- added C23: 2.2uF, Capacitor_SMD:C_0805_2012Metric_Pad1.15x1.40mm_HandSolder, F.Cu at (46.7, 65.0)
- added C24: 2.2uF, Capacitor_SMD:C_0805_2012Metric_Pad1.15x1.40mm_HandSolder, F.Cu at (41.9, 64.8)
- added C25: 2.2uF, Capacitor_SMD:C_0805_2012Metric_Pad1.15x1.40mm_HandSolder, F.Cu at (45.6, 37.6)
- added C26: 2.2uF, Capacitor_SMD:C_0805_2012Metric_Pad1.15x1.40mm_HandSolder, F.Cu at (37.1, 43.3)
- added D21: 1N4002, Diode_SMD:D_SOD-123F, F.Cu at (38.4, 38.4)
- added D22: 1N4002, Diode_SMD:D_SOD-123F, F.Cu at (37.5, 48.4)
- added D23: 12V Zener, Diode_SMD:D_SOD-123, F.Cu at (47.6, 40.7)
- added D24: 6.8V Zener, Diode_SMD:D_SOD-123, F.Cu at (53.1, 58.2)
- added J3: DEVHDR, Connector_PinSocket_2.54mm:PinSocket_2x05_P2.54mm_Vertical_SMD, F.Cu at (47.6, 49.2)
- added J5: VPPS, Jumper:SolderJumper-2_P1.3mm_Bridged_Pad1.0x1.5mm, F.Cu at (45.0, 85.5)
- added J7: VDDS, Jumper:SolderJumper-2_P1.3mm_Bridged_Pad1.0x1.5mm, F.Cu at (41.4, 85.0)
- added L3: 10uH, Inductor_SMD:L_2816_7142Metric, F.Cu at (48.1, 79.4)
- added L4: 10uH, Inductor_SMD:L_2816_7142Metric, F.Cu at (41.4, 78.9)
- added L5: 10uH, Inductor_SMD:L_2816_7142Metric, F.Cu at (40.3, 33.3)
- added L6: 10uH, Inductor_SMD:L_2816_7142Metric, F.Cu at (30.8, 39.7)
- added Q1: 3404, Package_TO_SOT_SMD:SOT-23, F.Cu at (49.3, 70.8)
- added Q2: 3404, Package_TO_SOT_SMD:SOT-23, F.Cu at (42.9, 70.8)
- added R10: 680, Resistor_SMD:R_0805_2012Metric_Pad1.15x1.40mm_HandSolder, F.Cu at (48.4, 60.8)
- added R11: 220, Resistor_SMD:R_0805_2012Metric_Pad1.15x1.40mm_HandSolder, F.Cu at (50.8, 65.1)
- added R12: 680, Resistor_SMD:R_0805_2012Metric_Pad1.15x1.40mm_HandSolder, F.Cu at (41.8, 55.3)
- added R13: 220, Resistor_SMD:R_0805_2012Metric_Pad1.15x1.40mm_HandSolder, F.Cu at (43.6, 60.0)
- R3: value 4.7k -> 4.7k-1%
- moved C18 46.2 mm to (86.1, 56.7), turned to 145 degrees
- moved R4 42.1 mm to (83.7, 59.7), turned to 255 degrees
- moved R6 41.0 mm to (82.7, 54.8), turned to 155 degrees
- moved MIC1 40.9 mm to (87.7, 60.6), turned to 180 degrees
- moved C16 34.4 mm to (81.3, 60.2), turned to 262.5 degrees
- moved R7 29.6 mm to (77.1, 55.9)
- moved R8 29.2 mm to (73.2, 59.3)
- moved R9 29.2 mm to (78.8, 59.5)
- moved U5 29.2 mm to (76.1, 59.5)
- moved J6 15.5 mm to (70.2, 56.1), turned to 0 degrees
Connections:
- net PA1 renamed PA2
- net PA3 renamed PA4
- U1 pad 10: Net-(U1-Pad10) -> A4
- U1 pad 11: Net-(U1-Pad11) -> VMON1
- U1 pad 12: ANA_ADC -> VMON2
- U1 pad 6: A0 -> ANA_ADC
- U1 pad 7: A1 -> TIM2_CH2
Routing:
- net GND: track 639.5 -> 863.0 mm, vias 23 -> 52
- net A4: track 0.00 -> 53.8 mm, vias 0 -> 2
- net TIM2_CH2: track 0.00 -> 38.0 mm, vias 0 -> 2
- net PD_VPP: track 0.00 -> 35.4 mm, vias 0 -> 2
- net Net-(C23-Pad1): track 0.00 -> 35.0 mm, vias 0 -> 2
- net PF0: track 0.00 -> 31.4 mm
- net SWC_TX: track 10.7 -> 41.3 mm, vias 0 -> 4
- net VUSB: track 75.8 -> 104.7 mm, vias 2 -> 5
- net PF1: track 0.00 -> 28.1 mm
- net Net-(C24-Pad1): track 0.00 -> 27.8 mm
- net AVCC: track 61.8 -> 34.0 mm, vias 3 -> 2
- net PD_VDD: track 0.00 -> 26.6 mm
- net A3: track 25.2 -> 49.3 mm, vias 2 -> 3
- net A1: track 22.8 -> 0.00 mm
- net VMON1: track 0.00 -> 22.5 mm
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- added copper zone on F.Cu, net A4
- removed copper zone on F.Cu, net A0
- removed copper zone on F.Cu, net A1
Other:
- board text removed: "#"
