File: attic/old_tensigral_lamp_2/tensigral_lamp_hardware.sch (KiCad schematic (older format))
At the start: 75 parts, among them J1 USB_B_Micro, J2 JTAG, J4 WSOUT, J6 MICJ, J8 WS_SEL, P1 WSIN, P10 AUXTOUCH, P2 WSOUT, P3 VLED, P4 VLED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

Commit message: Bump
Parts:
- removed C20: 22nF, Capacitor_SMD:C_0805_2012Metric_Pad1.15x1.40mm_HandSolder, symbol tensigral_lamp_hardware-rescue:C-Device-tensigral_lamp_hardware-rescue
- added C23, C24, C25, C26: 2.2uF, Capacitor_SMD:C_0805_2012Metric_Pad1.15x1.40mm_HandSolder, symbol tensigral_lamp_hardware-rescue:C-Device-tensigral_lamp_hardware-rescue
- added D21, D22: 1N4002, Diode_SMD:D_SOD-123F, symbol Device:D
- added D23: 12V Zener, Diode_SMD:D_SOD-123, symbol Device:D_Zener
- added D24: 6.8V Zener, Diode_SMD:D_SOD-123, symbol Device:D_Zener
- added J3: DEVHDR, Connector_PinSocket_2.54mm:PinSocket_2x05_P2.54mm_Vertical_SMD, symbol Connector_Generic:Conn_02x05_Odd_Even
- added J5: VPPS, Jumper:SolderJumper-2_P1.3mm_Bridged_Pad1.0x1.5mm, symbol Connector_Generic:Conn_01x02
- added J7: VDDS, Jumper:SolderJumper-2_P1.3mm_Bridged_Pad1.0x1.5mm, symbol Connector_Generic:Conn_01x02
- added L3, L4, L5, L6: 10uH, Inductor_SMD:L_2816_7142Metric, symbol tensigral_lamp_hardware-rescue:L-Device-tensigral_lamp_hardware-rescue
- added Q1, Q2: 3404, Package_TO_SOT_SMD:SOT-23, symbol Device:Q_NMOS_GSD
- added R10, R12: 680, Resistor_SMD:R_0805_2012Metric_Pad1.15x1.40mm_HandSolder, symbol tensigral_lamp_hardware-rescue:R-Device-tensigral_lamp_hardware-rescue
- added R11, R13: 220, Resistor_SMD:R_0805_2012Metric_Pad1.15x1.40mm_HandSolder, symbol tensigral_lamp_hardware-rescue:R-Device-tensigral_lamp_hardware-rescue
- R3: value 4.7k -> 4.7k-1%
Connections:
- net A0 is gone; now on net ANA_ADC: U1.6 (PA0)
- net A3: now also J3.5 (Pin_5)
- net ANA_ADC: no longer U1.12 (PA6)
- net GND: now also C25.2, C26.2, D23.2 (A), D24.2 (A), J3.2 (Pin_2), J3.4 (Pin_4), L5.2, L6.2, Q1.2 (S), Q2.2 (S), R11.1, R13.1
- net PF0: now also J3.8 (Pin_8)
- net PF1: now also J3.6 (Pin_6)
- net SWC_TX: now also J3.7 (Pin_7)
- net TIM3_CH4: now also Q1.1 (G)
- net VUSB: now also J3.1 (Pin_1), J5.1 (Pin_1), J7.1 (Pin_1)
- net A4: now reaches U1.10 (PA4)
- net A4: now also J3.10 (Pin_10)
- net VMON1: now reaches U1.11 (PA5)
- net VMON1: now also R12.1, R13.2
- net A1 renamed TIM2_CH2
- net TIM2_CH2: now also Q2.1 (G)
- net PA1 renamed PA2
- net PA3 renamed PA4
- new net: J5.2 (Pin_2), L3.1
- new net: C23.2, L3.2, Q1.3 (D)
- new net: C23.1, D21.2 (A), L5.1
- new net: J7.2 (Pin_2), L4.1
- new net: C24.2, L4.2, Q2.3 (D)
- new net: C24.1, D22.2 (A), L6.1
- new net PD_VDD: C26.1, D22.1 (K), D24.1 (K), J3.3 (Pin_3), R12.2
- new net PD_VPP: C25.1, D21.1 (K), D23.1 (K), J3.9 (Pin_9), R10.2
- new net VMON2: R10.1, R11.2, U1.12 (PA6)
Other:
- note added: "IPCK / U2CK\n"
- note added: "IPDA / U2TX"
- note added: "TODO: Can R6 be shorted?"
- note added: "U2RX"
- moved on the sheet: C19, R8, U4
