File: attic/old_tensigral_lamp_2/sepic_sim/sepic_sim.sch (KiCad schematic (older format))
At the start: 10 parts

Commit message: Bump
Parts:
- added Cmid?: C, symbol pspice:C
- Cmid: Spice_Model 1u -> 2.2u
- Rsource: Spice_Model .1 -> .2
- Vpulse: Spice_Model dc 10 pulse(0 10 0u 100n 100n 3u 5u) -> dc 10 pulse(0 10 0u 100n 100n 1500n 3u)
Connections:
- net 0: now also Cmid?.1
- net at Q?.1 (D), Rsource.2: now also Cmid?.2
Other:
- moved on the sheet: Rsource
Changed lines of the file:
@@
-$EndComp
-$Comp
-L pspice:C Cmid
-U 1 1 5EC9E1D7
-P 4150 2350
-F 0 "Cmid" V 3835 2350 50  0000 C CNN
-F 1 "C" V 3926 2350 50  0000 C CNN
-F 2 "" H 4150 2350 50  0001 C CNN
-F 3 "~" H 4150 2350 50  0001 C CNN
-F 4 "C" H 4150 2350 50  0001 C CNN "Spice_Primitive"
-F 5 "1u" H 4150 2350 50  0001 C CNN "Spice_Model"
-F 6 "Y" H 4150 2350 50  0001 C CNN "Spice_Netlist_Enabled"
-	1    4150 2350
-	0    1    1    0
 $EndComp
 $Comp
@@
 Wire Wire Line
 	2800 2450 2800 2350
-Wire Wire Line
-	2800 2350 3200 2350
 $Comp
 L Device:Q_NMOS_DGS Q?
@@
 P 3700 3300
 F 0 "Q?" H 3904 3346 50  0000 L CNN
-F 1 "Q_NMOS_DGS" H 3904 3255 50  0000 L CNN
+F 1 "Q_NMOS_DGS" H 3200 3450 50  0000 L CNN
 F 2 "" H 3900 3400 50  0001 C CNN
 F 3 "~" H 3700 3300 50  0001 C CNN
@@
 Wire Wire Line
 	3800 3500 3800 3700
-Wire Wire Line
-	3800 2600 3800 2350
-Wire Wire Line
-	3800 2350 3700 2350
-Wire Wire Line
-	3900 2350 3800 2350
-Connection ~ 3800 2350
 $Comp
 L pspice:INDUCTOR Lout
@@
 Wire Wire Line
 	4450 3200 4450 3050
-Wire Wire Line
-	4450 2550 4450 2350
-Wire Wire Line
-	4450 2350 4400 2350
 $Comp
 L pspice:VSOURCE Vpulse
@@
 F 3 "~" H 3450 4050 50  0001 C CNN
 F 4 "V" H 3450 4050 50  0001 C CNN "Spice_Primitive"
-F 5 "dc 10 pulse(0 10 0u 100n 100n 3u 5u)" H 3450 4050 50  0001 C CNN "Spice_Model"
+F 5 "dc 10 pulse(0 10 0u 100n 100n 1500n 3u)" H 3450 4050 50  0001 C CNN "Spice_Model"
 F 6 "Y" H 3450 4050 50  0001 C CNN "Spice_Netlist_Enabled"
 	1    3450 4050
@@
 Wire Wire Line
 	5200 3050 5200 3200
-Wire Wire Line
-	5200 2550 5200 2350
 $Comp
 L pspice:C Cout
@@
 Wire Wire Line
 	5550 2550 5550 2350
+$Comp
+L pspice:R Rsource
+U 1 1 5ECA420F
+P 3800 2750
+F 0 "Rsource" H 3868 2796 50  0000 L CNN
+F 1 "R" H 3868 2705 50  0000 L CNN
+F 2 "" H 3800 2750 50  0001 C CNN
+F 3 "~" H 3800 2750 50  0001 C CNN
+F 4 "R" H 3800 2750 50  0001 C CNN "Spice_Primitive"
+F 5 ".2" H 3800 2750 50  0001 C CNN "Spice_Model"
+F 6 "Y" H 3800 2750 50  0001 C CNN "Spice_Netlist_Enabled"
+	1    3800 2750
+	1    0    0    -1
+$EndComp
+Wire Wire Line
+	2800 2350 3200 2350
+Wire Wire Line
+	5200 2350 5550 2350
+Connection ~ 5200 2350
+Wire Wire Line
+	5000 2350 5200 2350
+Connection ~ 4450 2350
+Wire Wire Line
+	4600 2350 4450 2350
 $Comp
 L pspice:DIODE Drect
@@
 $EndComp
 Wire Wire Line
-	4600 2350 4450 2350
-Connection ~ 4450 2350
-Wire Wire Line
-	5000 2350 5200 2350
-Connection ~ 5200 2350
-Wire Wire Line
-	5200 2350 5550 2350
-$Comp
-L pspice:R Rsource
-U 1 1 5ECA420F
-P 3800 2850
-F 0 "Rsource" H 3868 2896 50  0000 L CNN
-F 1 "R" H 3868 2805 50  0000 L CNN
-F 2 "" H 3800 2850 50  0001 C CNN
-F 3 "~" H 3800 2850 50  0001 C CNN
-F 4 "R" H 3800 2850 50  0001 C CNN "Spice_Primitive"
-F 5 ".1" H 3800 2850 50  0001 C CNN "Spice_Model"
-F 6 "Y" H 3800 2850 50  0001 C CNN "Spice_Netlist_Enabled"
-	1    3800 2850
-	1    0    0    -1
-$EndComp
+	5200 2550 5200 2350
+Wire Wire Line
+	4450 2350 4400 2350
+Wire Wire Line
+	4450 2550 4450 2350
+$Comp
+L pspice:C Cmid
+U 1 1 5EC9E1D7
+P 4150 2350
+F 0 "Cmid" V 3835 2350 50  0000 C CNN
+F 1 "C" V 3926 2350 50  0000 C CNN
+F 2 "" H 4150 2350 50  0001 C CNN
+F 3 "~" H 4150 2350 50  0001 C CNN
+F 4 "C" H 4150 2350 50  0001 C CNN "Spice_Primitive"
+F 5 "2.2u" H 4150 2350 50  0001 C CNN "Spice_Model"
+F 6 "Y" H 4150 2350 50  0001 C CNN "Spice_Netlist_Enabled"
+	1    4150 2350
+	0    1    1    0
+$EndComp
+$Comp
+L pspice:C Cmid?
+U 1 1 5ECBC084
+P 4150 3350
+F 0 "Cmid?" V 3835 3350 50  0000 C CNN
+F 1 "C" V 3926 3350 50  0000 C CNN
+F 2 "" H 4150 3350 50  0001 C CNN
+F 3 "~" H 4150 3350 50  0001 C CNN
+F 4 "C" H 4150 3350 50  0001 C CNN "Spice_Primitive"
+F 5 "600p" H 4150 3350 50  0001 C CNN "Spice_Model"
+F 6 "Y" H 4150 3350 50  0001 C CNN "Spice_Netlist_Enabled"
+	1    4150 3350
+	-1   0    0    1
+$EndComp
+Wire Wire Line
+	3700 2350 3800 2350
+Wire Wire Line
+	3800 3000 3800 3050
+Wire Wire Line
+	3800 3050 4150 3050
+Wire Wire Line
+	4150 3050 4150 3100
+Connection ~ 3800 3050
+Wire Wire Line
+	3800 3050 3800 3100
+Wire Wire Line
+	3800 2500 3800 2350
+Connection ~ 3800 2350
+Wire Wire Line
+	3800 2350 3900 2350
+$Comp
+L pspice:0 #GND?
+U 1 1 5ECBFF1F
+P 4150 3700
+F 0 "#GND?" H 4150 3600 50  0001 C CNN
+F 1 "0" H 4150 3789 50  0000 C CNN
+F 2 "" H 4150 3700 50  0001 C CNN
+F 3 "~" H 4150 3700 50  0001 C CNN
+	1    4150 3700
+	1    0    0    -1
+$EndComp
+Wire Wire Line
+	4150 3700 4150 3600
 $EndSCHEMATC
