File: tensigral_lamp_2/tensigral_lamp_hardware.kicad_pcb (KiCad board)
At the start: 2 copper layers, 99.5 x 99.8 mm, 69 parts, among them J1 USB_B_Micro, J2 JTAG, J3 EXTCTL, J4 WSOUT, J5 AVRISP6, P1 WSIN, P10 AUXOUT, P11 AUXEXTRA, P2 WSOUT, P3 VLED, P4 VLED, P5 GND, P6 GND, P7 AUX, P8 WS, P9 AUXOUT, SW1 TACTILE, T0 TOUCH0, T1 TOUCH1, T2 TOUCH2, U1 STM32F042F4Px, U2 MT2492, U3 ATtiny45-20SU, U4 MXC400xXC

Commit message: Bump
Parts:
- removed MK1: Microphone, kicad:9mmELECTRET_MIC_SMT
- removed P11: AUXEXTRA, Connector_Wire:SolderWirePad_1x01_Drill1mm
- removed P7: AUX, Connector_Wire:SolderWirePad_1x01_Drill0.8mm
- removed P8: WS, Connector_Wire:SolderWirePad_1x01_Drill0.8mm
- removed R5: 6.8k-1%, Resistor_SMD:R_0805_2012Metric_Pad1.15x1.40mm_HandSolder
- added C18: 2.2uF, Capacitor_SMD:C_0805_2012Metric_Pad1.15x1.40mm_HandSolder, F.Cu at (86.1, 56.7)
- added C19: 2.2uF, Capacitor_SMD:C_0805_2012Metric_Pad1.15x1.40mm_HandSolder, F.Cu at (64.4, 63.3)
- added C22: 22uF, Capacitor_SMD:C_0805_2012Metric_Pad1.15x1.40mm_HandSolder, F.Cu at (107.9, 48.1)
- added C23: 2.2uF, Capacitor_SMD:C_0805_2012Metric_Pad1.15x1.40mm_HandSolder, F.Cu at (46.7, 65.0)
- added C24: 2.2uF, Capacitor_SMD:C_0805_2012Metric_Pad1.15x1.40mm_HandSolder, F.Cu at (41.9, 64.8)
- added C25: 2.2uF, Capacitor_SMD:C_0805_2012Metric_Pad1.15x1.40mm_HandSolder, F.Cu at (45.6, 37.6)
- added C26: 2.2uF, Capacitor_SMD:C_0805_2012Metric_Pad1.15x1.40mm_HandSolder, F.Cu at (37.1, 43.3)
- added D21: 1N4002, Diode_SMD:D_SOD-123F, F.Cu at (38.4, 38.4)
- added D22: 1N4002, Diode_SMD:D_SOD-123F, F.Cu at (37.5, 48.4)
- added D23: 12V Zener, Diode_SMD:D_SOD-123, F.Cu at (47.6, 40.7)
- added D24: 6.8V Zener, Diode_SMD:D_SOD-123, F.Cu at (53.1, 58.2)
- added J6: MICJ, Jumper:SolderJumper-2_P1.3mm_Bridged_Pad1.0x1.5mm, F.Cu at (70.2, 56.1)
- added J7: VDDS, Jumper:SolderJumper-2_P1.3mm_Bridged_Pad1.0x1.5mm, F.Cu at (41.4, 85.0)
- added J8: WS_SEL, Jumper:SolderJumper-2_P1.3mm_Bridged_Pad1.0x1.5mm, F.Cu at (88.0, 70.5)
- added L2: 10uH, Inductor_SMD:L_2816_7142Metric, F.Cu at (75.5, 65.7)
- added L3: 10uH, Inductor_SMD:L_2816_7142Metric, F.Cu at (48.1, 79.4)
- added L4: 10uH, Inductor_SMD:L_2816_7142Metric, F.Cu at (41.4, 78.9)
- added L5: 10uH, Inductor_SMD:L_2816_7142Metric, F.Cu at (40.3, 33.3)
- added L6: 10uH, Inductor_SMD:L_2816_7142Metric, F.Cu at (30.8, 39.7)
- added MIC1: ZTS6011E, ZTS6011E-MICROPHONE:ZTS6011E, F.Cu at (87.7, 60.6)
- added Q1: 3404, Package_TO_SOT_SMD:SOT-23, F.Cu at (49.3, 70.8)
- added Q2: 3404, Package_TO_SOT_SMD:SOT-23, F.Cu at (42.9, 70.8)
- added R10: 680, Resistor_SMD:R_0805_2012Metric_Pad1.15x1.40mm_HandSolder, F.Cu at (48.4, 60.8)
- added R11: 220, Resistor_SMD:R_0805_2012Metric_Pad1.15x1.40mm_HandSolder, F.Cu at (50.8, 65.1)
- added R12: 680, Resistor_SMD:R_0805_2012Metric_Pad1.15x1.40mm_HandSolder, F.Cu at (41.8, 55.3)
- added R13: 220, Resistor_SMD:R_0805_2012Metric_Pad1.15x1.40mm_HandSolder, F.Cu at (43.6, 60.0)
- added R7: 27k, Resistor_SMD:R_0805_2012Metric_Pad1.15x1.40mm_HandSolder, F.Cu at (77.1, 55.9)
- added R8: 220k, Resistor_SMD:R_0805_2012Metric_Pad1.15x1.40mm_HandSolder, F.Cu at (73.2, 59.3)
- added R9: 27k, Resistor_SMD:R_0805_2012Metric_Pad1.15x1.40mm_HandSolder, F.Cu at (78.8, 59.5)
- added T1: TOUCH1, kicad:TOUCH_MARK, F.Cu at (74.3, 105.1)
- added U5: LM321, Package_TO_SOT_SMD:SOT-23-5, F.Cu at (76.1, 59.5)
- J3: value EXTCTL -> DEVHDR; footprint kicad:RIBBON6SMT_POGO_OR_IDC -> Connector_PinSocket_2.54mm:PinSocket_2x05_P2.54mm_Vertical_SMD
- J5: value AVRISP6 -> VPPS; footprint kicad:RIBBON6SMT_POGO_OR_IDC -> Jumper:SolderJumper-2_P1.3mm_Bridged_Pad1.0x1.5mm
- P10: value AUXOUT -> AUXTOUCH
- P9: value AUXOUT -> TOPTOUCH
- R1: value 33k-1% -> 27k
- R2, R4, R6: value 6.8k-1% -> 4.7k
- R3: value 6.8k-1% -> 4.7k-1%
- SW1: value TACTILE -> BOOT0
- T2: renamed from T1; value TOUCH1 -> TOUCH2; moved to B.Cu
- TOUCH1: renamed from T0; value TOUCH0 -> TA3
- TOUCH2: renamed from T2; value TOUCH2 -> TA3; moved to B.Cu
- U3: value ATtiny45-20SU -> NUP4202; footprint Package_SO:SOIJ-8_5.3x5.3mm_P1.27mm -> Package_TO_SOT_SMD:SOT-363_SC-70-6
- U4: value MXC400xXC -> XC6206P360MR; footprint kicad:MXC400xXC -> Package_TO_SOT_SMD:SOT-23
- moved P5 85.1 mm to (27.0, 108.0)
- moved P3 84.8 mm to (26.8, 22.9)
- moved T2 77.4 mm to (74.3, 105.2)
- moved TOUCH1 71.2 mm to (83.4, 35.7)
- moved P4 60.8 mm to (33.8, 95.8)
- moved J5 60.6 mm to (45.0, 85.5), turned to 60 degrees
- moved P6 60.6 mm to (33.8, 35.1)
- moved U3 56.9 mm to (54.6, 79.4), turned to 90 degrees
- moved P9 56.7 mm to (70.2, 35.3), turned to 42 degrees
- moved R6 56.0 mm to (82.7, 54.8), turned to 155 degrees
- moved U4 52.2 mm to (57.8, 66.9), turned to 250 degrees
- moved C17 42.8 mm to (69.5, 62.7), turned to 255 degrees
- moved J3 25.8 mm to (47.6, 49.2), turned to 210 degrees
- moved J1 25.2 mm to (49.9, 91.6), turned to 58 degrees
- moved TOUCH2 22.8 mm to (83.5, 35.7)
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Connections:
- C12 pad 1: +3V8 -> VLED
- C16 pad 1: AUXVCC -> AVCC
- C16 pad 2: AUXGND -> GND
- C17 pad 1: AUXVCC -> AVCC
- C17 pad 2: AUXGND -> GND
- C9 pad 1: +3V8 -> VLED
- D3 pad 2: (no net) -> Net-(D3-Pad2)
- J1 pad 4: (no net) -> Net-(J1-Pad4)
- J2 pad 3: SWC -> SWC_TX
- J2 pad 4: (no net) -> Net-(J2-Pad4)
- J3 pad 1: PA4 -> VUSB
- J3 pad 2: PF1 -> GND
- J3 pad 3: PA5 -> PD_VDD
- J3 pad 4: PF0 -> GND
- J3 pad 5: PA6 -> A3
- J3 pad 6: GND -> PF1
- J4 pad 2: WS2812U -> WS2812
- J5 pad 1: Net-(J5-Pad1) -> VUSB
- J5 pad 2: AUXVCC -> Net-(J5-Pad2)
- L1 pad 2: +3V8 -> VLED
- P4 pad 1: +3V8 -> VLED
- P9 pad 1: AUXU -> TTVAL
- R1 pad 2: +3V8 -> VLED
- R4 pad 1: ASDA -> Net-(C18-Pad1)
- R4 pad 2: AUXVCC -> AVCC
- R6 pad 1: ANA_ADC -> Net-(C18-Pad2)
- R6 pad 2: +3V8 -> Net-(R6-Pad2)
- SW1 pad 1: +3V8 -> VLED
- SW1 pad 2: (no net) -> Net-(SW1-Pad2)
- SW1 pad 3: (no net) -> Net-(SW1-Pad3)
- T2 pad 1: Net-(T1-Pad1) -> PA2
- TOUCH1 pad 1: Net-(T0-Pad1) -> TTVAL
- TOUCH2 pad 1: Net-(T2-Pad1) -> TTVAL
- U1 pad 10: PA4 -> A4
- U1 pad 11: PA5 -> VMON1
- U1 pad 12: PA6 -> VMON2
- U1 pad 13: WS2812U -> WS2812
- U1 pad 14: AUX -> TIM3_CH4
- U1 pad 16: +3V8 -> +3V3
- U1 pad 20: SWC -> SWC_TX
- U1 pad 5: +3V8 -> AVCC
- U1 pad 6: Net-(T0-Pad1) -> ANA_ADC
- U1 pad 7: Net-(T1-Pad1) -> TIM2_CH2
- U1 pad 8: ANA_ADC -> A2
- U1 pad 9: Net-(T2-Pad1) -> A3
- U3 pad 1: Net-(J5-Pad5) -> D-
- U3 pad 2: ASDA -> GND
- U3 pad 3: ASCL -> D+
- U3 pad 4: AUXGND -> D+
- U3 pad 5: AUXEXTRA -> VUSB
- U3 pad 6: Net-(J5-Pad1) -> D-
- U4 pad 1: ASCL -> GND
- U4 pad 2: (no net) -> +3V3
- U4 pad 3: AUXGND -> VLED
Routing:
- net GND: track 544.1 -> 863.0 mm, vias 14 -> 52
- net VLED: track 288.0 -> 429.7 mm, vias 0 -> 2
- net +3V8: track 107.9 -> 0.00 mm, vias 4 -> 0
- net WS2812U: track 76.4 -> 0.00 mm, vias 2 -> 0
- net AUXGND: track 69.8 -> 2.12 mm, vias 6 -> 1
- net Net-(T0-Pad1): track 55.7 -> 0.00 mm, vias 4 -> 0
- net AUXVCC: track 56.3 -> 2.24 mm, vias 3 -> 1
- net A4: track 0.00 -> 53.8 mm, vias 0 -> 2
- net WS2812: track 5.66 -> 58.5 mm, vias 0 -> 4
- net ANA_ADC: track 56.9 -> 4.38 mm
- net AUX: track 51.7 -> 0.00 mm, vias 2 -> 0
- net A3: track 0.00 -> 49.3 mm, vias 0 -> 3
- net SWC_TX: track 0.00 -> 41.3 mm, vias 0 -> 4
- net TIM2_CH2: track 0.00 -> 38.0 mm, vias 0 -> 2
- net Net-(T1-Pad1): track 36.3 -> 0.00 mm
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- added copper zone on F.Cu, net A2
- added copper zone on F.Cu, net A3
- added copper zone on F.Cu, net A4
- added copper zone on B.Cu, net PA2
- added copper zone on F.Cu, net PA2
- added copper zone on B.Cu, net PA4
- added copper zone on F.Cu, net PA4
- added copper zone on B.Cu, net TTVAL
- added copper zone on F.Cu, net TTVAL
- added copper zone on F.Cu, net WS2812STAFF
- removed copper zone on F.Cu, net (none)
- removed copper zone on F.Cu, net AUX
- removed copper zone on F.Cu, net WS2812U
Other:
- board size 99.5 x 99.8 mm -> 99 x 99.8 mm
- board text added: "*"
- board text added: "GND 2812 VUSB"
- board text added: "tensigral_lamp rev A https://github.com/cnlohr/tensigral_lamp"
- board text removed: "0V RST MO SK 4V MI"
- board text removed: "PA4 PF1 PA5 PF0 PA6 GND"
- board text removed: "WS"
- board text removed: "tensigral_lamp r - https://github.com/cnlohr/tensigral_lamp"

Commit message: Bump
Parts:
- removed C23, C24, C25, C26: 2.2uF, Capacitor_SMD:C_0805_2012Metric_Pad1.15x1.40mm_HandSolder
- removed D21, D22: 1N4002, Diode_SMD:D_SOD-123F
- removed D23: 12V Zener, Diode_SMD:D_SOD-123
- removed D24: 6.8V Zener, Diode_SMD:D_SOD-123
- removed J3: DEVHDR, Connector_PinSocket_2.54mm:PinSocket_2x05_P2.54mm_Vertical_SMD
- removed J5: VPPS, Jumper:SolderJumper-2_P1.3mm_Bridged_Pad1.0x1.5mm
- removed J7: VDDS, Jumper:SolderJumper-2_P1.3mm_Bridged_Pad1.0x1.5mm
- removed L3, L4, L5, L6: 10uH, Inductor_SMD:L_2816_7142Metric
- removed Q1, Q2: 3404, Package_TO_SOT_SMD:SOT-23
- removed R10, R12: 680, Resistor_SMD:R_0805_2012Metric_Pad1.15x1.40mm_HandSolder
- removed R11, R13: 220, Resistor_SMD:R_0805_2012Metric_Pad1.15x1.40mm_HandSolder
- added C20: 22nF, Capacitor_SMD:C_0805_2012Metric_Pad1.15x1.40mm_HandSolder, F.Cu at (42.6, 64.8)
- R3: value 4.7k-1% -> 4.7k
- moved C18 46.2 mm to (39.9, 54.3), turned to 295 degrees
- moved R4 42.1 mm to (42.6, 50.4), turned to 345 degrees
- moved R6 41.0 mm to (41.8, 58.4), turned to 275 degrees
- moved MIC1 40.9 mm to (47.1, 55.5), turned to 0 degrees
- moved C16 34.4 mm to (48.2, 50.9), turned to 0 degrees
- moved R7 29.6 mm to (48.0, 61.6)
- moved R8 29.2 mm to (44.5, 64.8)
- moved R9 29.2 mm to (50.1, 65.0)
- moved U5 29.2 mm to (47.4, 65.0)
- moved J6 15.5 mm to (55.1, 59.7), turned to 210 degrees
- moved U3 2.30 mm to (52.3, 79.2), turned to 60 degrees
- moved J1 0.14 mm to (50.0, 91.7)
Connections:
- net PA2 renamed PA1
- net PA4 renamed PA3
- U1 pad 10: A4 -> Net-(U1-Pad10)
- U1 pad 11: VMON1 -> Net-(U1-Pad11)
- U1 pad 12: VMON2 -> ANA_ADC
- U1 pad 6: ANA_ADC -> A0
- U1 pad 7: TIM2_CH2 -> A1
Routing:
- net GND: track 863.0 -> 633.2 mm, vias 52 -> 24
- net A4: track 53.8 -> 0.00 mm, vias 2 -> 0
- net TIM2_CH2: track 38.0 -> 0.00 mm, vias 2 -> 0
- net PD_VPP: track 35.4 -> 0.00 mm, vias 2 -> 0
- net Net-(C23-Pad1): track 35.0 -> 0.00 mm, vias 2 -> 0
- net PF0: track 31.4 -> 0.00 mm
- net SWC_TX: track 41.3 -> 10.7 mm, vias 4 -> 0
- net PF1: track 28.1 -> 0.00 mm
- net Net-(C24-Pad1): track 27.8 -> 0.00 mm
- net AVCC: track 34.0 -> 61.8 mm, vias 2 -> 3
- net VUSB: track 104.7 -> 77.3 mm, vias 5 -> 2
- net PD_VDD: track 26.6 -> 0.00 mm
- net A3: track 49.3 -> 25.2 mm, vias 3 -> 2
- net A1: track 0.00 -> 22.8 mm
- net VMON1: track 22.5 -> 0.00 mm
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- added copper zone on F.Cu, net A0
- added copper zone on F.Cu, net A1
- removed copper zone on F.Cu, net A4
Other:
- board text added: "#"
