File: tensigral_lamp_2/tensigral_lamp_hardware.sch (KiCad schematic (older format))
At the start: 85 parts, among them J1 USB_B_Micro, J2 JTAG, J4 WSOUT, P1 WSIN, P10 AUXOUT, P2 WSOUT, P3 VLED, P4 VLED, P5 GND, P6 GND, P7 AUX, P8 WS, P9 AUXOUT, SW1 TACTILE, T0 TOUCH0, T1 TOUCH1, T2 TOUCH2, U1 STM32F042F4Px, U2 MT2492

Commit message: Bump
Parts:
- removed C? (x2): 2.2uF/25v, Capacitor_SMD:C_0805_2012Metric_Pad1.15x1.40mm_HandSolder, symbol tensigral_lamp_hardware-rescue:C-Device-tensigral_lamp_hardware-rescue
- removed MK1: Microphone, kicad:9mmELECTRET_MIC_SMT, symbol tensigral_lamp_hardware-rescue:Microphone-Device-tensigral_lamp_hardware-rescue
- removed P7: AUX, Connector_Wire:SolderWirePad_1x01_Drill0.8mm, symbol tensigral_lamp_hardware-rescue:CONN_1-5050RGB-tensigral_lamp_hardware-rescue
- removed P8: WS, Connector_Wire:SolderWirePad_1x01_Drill0.8mm, symbol tensigral_lamp_hardware-rescue:CONN_1-5050RGB-tensigral_lamp_hardware-rescue
- added C18: 2.2uF, Capacitor_SMD:C_0805_2012Metric_Pad1.15x1.40mm_HandSolder, symbol tensigral_lamp_hardware-rescue:C-Device-tensigral_lamp_hardware-rescue
- added D23: 12V Zener, Diode_SMD:D_SOD-123, symbol Device:D_Zener
- added D24: 6.8V Zener, Diode_SMD:D_SOD-123, symbol Device:D_Zener
- added J5: VPPS, Jumper:SolderJumper-2_P1.3mm_Bridged_Pad1.0x1.5mm, symbol Connector_Generic:Conn_01x02
- added J6: MICJ, Jumper:SolderJumper-2_P1.3mm_Bridged_Pad1.0x1.5mm, symbol Connector_Generic:Conn_01x02
- added J7: VDDS, Jumper:SolderJumper-2_P1.3mm_Bridged_Pad1.0x1.5mm, symbol Connector_Generic:Conn_01x02
- added J8: WS_SEL, Jumper:SolderJumper-2_P1.3mm_Bridged_Pad1.0x1.5mm, symbol Connector_Generic:Conn_01x02
- added MIC1: ZTS6011E, ZTS6011E-MICROPHONE:ZTS6011E, symbol Connector_Generic:Conn_01x04
- added R4: 4.7k, Resistor_SMD:R_0805_2012Metric_Pad1.15x1.40mm_HandSolder, symbol tensigral_lamp_hardware-rescue:R-Device-tensigral_lamp_hardware-rescue
- added R7, R9: 27k, Resistor_SMD:R_0805_2012Metric_Pad1.15x1.40mm_HandSolder, symbol tensigral_lamp_hardware-rescue:R-Device-tensigral_lamp_hardware-rescue
- added R8: 220k, Resistor_SMD:R_0805_2012Metric_Pad1.15x1.40mm_HandSolder, symbol tensigral_lamp_hardware-rescue:R-Device-tensigral_lamp_hardware-rescue
- added TOUCH1: TA3, kicad:TOUCH_MARK, symbol tensigral_lamp_hardware-rescue:CONN_1-5050RGB-tensigral_lamp_hardware-rescue
- added U3: NUP4202, Package_TO_SOT_SMD:SOT-363_SC-70-6, symbol Power_Protection:NUP4202
- added U5: LM321, Package_TO_SOT_SMD:SOT-23-5, symbol Amplifier_Operational:LM321
- C19, C23, C24, C25, C26: renamed from C?; value 2.2uF/25v -> 2.2uF
- J3: renamed from J?; value Conn_02x05_Odd_Even -> DEVHDR; footprint (none) -> Connector_PinSocket_2.54mm:PinSocket_2x05_P2.54mm_Vertical_SMD
- P10: value AUXOUT -> AUXTOUCH
- P9: value AUXOUT -> TOPTOUCH
- R1: value 27k-1% -> 27k
- R2: value 4.7k-1% -> 4.7k
- R6: value 6.8k-1% -> 4.7k; Cost100 .00104 -> 0.002315; LCSC https://lcsc.com/product-detail/Chip-Resistor-Surface-Mount_UNI-ROYAL-Uniroyal-Elec-0805W8F6801T5E_C17772.html -> https://lcsc.com/product-detail/Chip-Resistor-Surface-Mount_UNI-ROYAL-Uniroyal-Elec-0805W8F4701T5E_C17673.html
- SW1: value TACTILE -> BOOT0
- TOUCH2: renamed from T0; value TOUCH0 -> TA3
- U4: renamed from U?; value XC6206PxxxMR -> XC6206P360MR; Cost100 (none) -> 0.017802; LCSC (none) -> https://lcsc.com/product-detail/Low-Dropout-Regulators-LDO_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
- gave numbers to parts that had none: 17
Connections:
- net SWC is gone; now on net SWC_TX: J2.3 (Pin_3)
- net WS2812U is gone; now on net WS2812: J4.2 (Pin_2), U1.13 (PA7)
- net +3V8: now also C1.1, C10.1, C2.1, C3.1, C4.1, C5.1, C6.1, C7.1, C8.1, D1.1 (VDD), D10.1 (VDD), D11.1 (VDD), D12.1 (VDD), D13.1 (VDD), D14.1 (VDD), D15.1 (VDD), D16.1 (VDD), D17.1 (VDD), D18.1 (VDD), D19.1 (VDD), D2.1 (VDD), D20.1 (VDD), D3.1 (VDD), D4.1 (VDD), D5.1 (VDD), D6.1 (VDD), D7.1 (VDD), D8.1 (VDD), D9.1 (VDD), P3.1; no longer R6.2
- net A2: no longer T2.1
- net A3: no longer TOUCH2.1
- net A4: no longer T1.1
- net ANA_ADC: now also J6.1 (Pin_1); no longer R6.1
- net AUXU: no longer P9.1
- net D+: now also U3.3, U3.4
- net D-: now also U3.1, U3.6
- net GND: now also D23.2 (A), D24.2 (A), MIC1.2 (Pin_2), MIC1.3 (Pin_3), R7.1, U3.2, U5.2 (V-); no longer C22.2
- net PD_VDD: now also D24.1 (K)
- net PD_VPP: now also D23.1 (K)
- net VUSB: now also J5.1 (Pin_1), J7.1 (Pin_1), U3.5; no longer L3.1, L4.1
- net WS2812: now also J8.1 (Pin_1)
- net AVCC: now reaches C16.1, C17.1, L2.2, U1.5 (VDDA)
- net AVCC: now also MIC1.1 (Pin_1), R4.2, R9.2, U5.5 (V+)
- removed net VLED: C1.1, C10.1, C2.1, C22.1, C3.1, C4.1, C5.1, C6.1, C7.1, C8.1, D1.1 (VDD), D10.1 (VDD), D11.1 (VDD), D12.1 (VDD), D13.1 (VDD), D14.1 (VDD), D15.1 (VDD), D16.1 (VDD), D17.1 (VDD), D18.1 (VDD), D19.1 (VDD), D2.1 (VDD), D20.1 (VDD), D3.1 (VDD), D4.1 (VDD), D5.1 (VDD), D6.1 (VDD), D7.1 (VDD), D8.1 (VDD), D9.1 (VDD), P3.1
- new net: J6.2 (Pin_2), R8.2, U5.4
- new net: C18.1, MIC1.4 (Pin_4), R4.1
- new net: C18.2, R6.1
- new net: J5.2 (Pin_2), L3.1
- new net: R6.2, R8.1, U5.3 (-)
- new net: R7.2, R9.1, U5.1 (+)
- new net: J7.2 (Pin_2), L4.1
- new net AUXGND: C22.2
- new net AUXVCC: C22.1
- new net PA2: T2.1
- new net PA4: T1.1
- new net TTVAL: P9.1, TOUCH1.1, TOUCH2.1
- new net WS2812STAFF: J8.2 (Pin_2)
Other:
- note added: "TODO: Can R6 be shorted?"
- note removed: "USB Protection\nATTiny / UPDI / PADAUK"
- moved on the sheet: C11, C12, C13, C14, C15, C19, C24, C26, C9, D22, J1, J3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

Commit message: Bump
Parts:
- removed C23, C24, C25, C26: 2.2uF, Capacitor_SMD:C_0805_2012Metric_Pad1.15x1.40mm_HandSolder, symbol tensigral_lamp_hardware-rescue:C-Device-tensigral_lamp_hardware-rescue
- removed D21, D22: 1N4002, Diode_SMD:D_SOD-123F, symbol Device:D
- removed D23: 12V Zener, Diode_SMD:D_SOD-123, symbol Device:D_Zener
- removed D24: 6.8V Zener, Diode_SMD:D_SOD-123, symbol Device:D_Zener
- removed J3: DEVHDR, Connector_PinSocket_2.54mm:PinSocket_2x05_P2.54mm_Vertical_SMD, symbol Connector_Generic:Conn_02x05_Odd_Even
- removed J5: VPPS, Jumper:SolderJumper-2_P1.3mm_Bridged_Pad1.0x1.5mm, symbol Connector_Generic:Conn_01x02
- removed J7: VDDS, Jumper:SolderJumper-2_P1.3mm_Bridged_Pad1.0x1.5mm, symbol Connector_Generic:Conn_01x02
- removed L3, L4, L5, L6: 10uH, Inductor_SMD:L_2816_7142Metric, symbol tensigral_lamp_hardware-rescue:L-Device-tensigral_lamp_hardware-rescue
- removed Q1, Q2: 3404, Package_TO_SOT_SMD:SOT-23, symbol Device:Q_NMOS_GSD
- removed R10, R12: 680, Resistor_SMD:R_0805_2012Metric_Pad1.15x1.40mm_HandSolder, symbol tensigral_lamp_hardware-rescue:R-Device-tensigral_lamp_hardware-rescue
- removed R11, R13: 220, Resistor_SMD:R_0805_2012Metric_Pad1.15x1.40mm_HandSolder, symbol tensigral_lamp_hardware-rescue:R-Device-tensigral_lamp_hardware-rescue
- added C20: 22nF, Capacitor_SMD:C_0805_2012Metric_Pad1.15x1.40mm_HandSolder, symbol tensigral_lamp_hardware-rescue:C-Device-tensigral_lamp_hardware-rescue
- R3: value 4.7k-1% -> 4.7k
Connections:
- net VMON2 is gone; now on net ANA_ADC: U1.12 (PA6)
- net ANA_ADC: no longer U1.6 (PA0)
- net at J6.2 (Pin_2), R8.2, U5.4: now also C20.1
- net at R6.2, R8.1, U5.3 (-): now also C20.2
- net A4: no longer names the net of U1.10 (PA4)
- net PA2 renamed PA1
- net PA4 renamed PA3
- net TIM2_CH2 renamed A1
- net VMON1: no longer names the net of U1.11 (PA5)
- new net A0: U1.6 (PA0)
Other:
- note added: "Differences:\n * Using opamp in microphone circuit\n * Putting touch on staff.\n * 90 degree mounting of inside strings.\n * Connecting LEDs before tear-apart for testing."
- note removed: "IPCK / U2CK\n"
- note removed: "IPDA / U2TX"
- note removed: "TODO: Can R6 be shorted?"
- note removed: "U2RX"
- moved on the sheet: C19, R8, U4
